File: color-swatches.kicad_pcb (KiCad board)
At the start: 2 copper layers, 89.6 x 94.6 mm, 6 parts

Commit message: updated to v1
Parts:
- removed the G*** at (0.00, 0.00) (x6)
- added G*** (x6): LOGO, LOGO, F.Cu at (0.00, 0.00)
